Commit message: fixed URDF to improved odometry

File: kachaka_description/urdf/_kachaka.urdf.xacro (robot description, xacro)
@@ -39,7 +39,7 @@
       <parent link="base_link" />
       <child link="base_r_drive_wheel_link" />
-      <origin rpy="0 0 0"
+      <origin rpy="-1.57 0 0"
               xyz="0.0 -0.100 0.045" />
-      <axis xyz="0 1 0" />
+      <axis xyz="0 0 1" />
     </joint>
     <link name="base_r_drive_wheel_link">
@@ -47,5 +47,5 @@
         <mass value="0.2" /> <!-- TODO - Update mass value -->
         <origin xyz="0 0 0"
-                rpy="${PI / 2.0} 0 0" />
+                rpy="-1.57 0 0" />
         <!-- Bug - inertial rotation is not reflected in Rviz2 -->
         <!-- https://github.com/ros2/rviz/pull/1316 -->
@@ -55,5 +55,5 @@
       </inertial>
       <visual>
-        <origin rpy="0 0 0" xyz="0 0 0"/>
+        <origin rpy="-1.57 0 0" xyz="0 0 0"/>
         <geometry>
           <mesh filename="package://kachaka_description/meshes/kachaka/right_tire.stl" scale="1.0 1.0 1.0"/>
@@ -63,5 +63,5 @@
       <collision>
         <origin xyz="0 0 0"
-                rpy="1.57079637 0 0" />
+                rpy="0 0 0" />
         <geometry>
           <cylinder length="0.025"
@@ -97,7 +97,7 @@
       <parent link="base_link" />
       <child link="base_l_drive_wheel_link" />
-      <origin rpy="0 0 0"
+      <origin rpy="-1.57 0 0"
               xyz="0.0 0.100 0.045" />
-      <axis xyz="0 1 0" />
+      <axis xyz="0 0 1" />
     </joint>
     <link name="base_l_drive_wheel_link">
@@ -105,5 +105,5 @@
         <mass value="0.2" />
         <origin xyz="0 0 0"
-                rpy="1.57079637 0 0" />
+                rpy="-1.57 0 0" />
         <!-- Bug - inertial rotation is not reflected in Rviz2 -->
         <!-- https://github.com/ros2/rviz/pull/1316 -->
@@ -114,5 +114,5 @@
       <visual>
         <origin xyz="0 0 0"
-                rpy="0 0 0" />
+                rpy="-1.57 0 0" />
         <geometry>
           <mesh filename="package://kachaka_description/meshes/kachaka/left_tire.stl" scale="1.0 1.0 1.0"/>
@@ -122,5 +122,5 @@
       <collision>
         <origin xyz="0 0 0"
-                rpy="1.57079637 0 0" />
+                rpy="0 0 0" />
         <geometry>
           <cylinder length="0.025"

Commit message: fixed URDF

File: kachaka_description/urdf/_kachaka.urdf.xacro (robot description, xacro)
@@ -12,5 +12,5 @@
       <inertial>
         <mass value="10.0" />
-        <origin xyz="0.0435 0.0 0.0475"
+        <origin xyz="0.0435 0.0 0.045"
                 rpy="0 0 0" />
         <inertia ixx="${1/12*10*(0.095**2+0.240**2)}" ixy="0" ixz="0"
@@ -26,5 +26,5 @@
       </visual>
       <collision>
-        <origin xyz="0.0435 0.0 0.0475"
+        <origin xyz="0.0435 0.0 0.045"
                 rpy="0 0 0" />
         <geometry>
@@ -40,5 +40,5 @@
       <child link="base_r_drive_wheel_link" />
       <origin rpy="-1.57 0 0"
-              xyz="0.0 -0.100 0.045" />
+              xyz="0.0 -0.100 0.04" />
       <axis xyz="0 0 1" />
     </joint>
@@ -66,5 +66,5 @@
         <geometry>
           <cylinder length="0.025"
-                    radius="0.0475" />
+                    radius="0.045" />
         </geometry>
         <material name="tire" />
@@ -98,5 +98,5 @@
       <child link="base_l_drive_wheel_link" />
       <origin rpy="-1.57 0 0"
-              xyz="0.0 0.100 0.045" />
+              xyz="0.0 0.100 0.04" />
       <axis xyz="0 0 1" />
     </joint>
@@ -125,5 +125,5 @@
         <geometry>
           <cylinder length="0.025"
-                    radius="0.0475" />
+                    radius="0.045" />
         </geometry>
         <material name="tire" />
@@ -158,5 +158,5 @@
           <right_joint>base_r_drive_wheel_joint</right_joint>
           <wheel_separation>0.2</wheel_separation>
-          <wheel_radius>0.0475</wheel_radius>
+          <wheel_radius>0.045</wheel_radius>
           <max_linear_acceleration>2</max_linear_acceleration>
           <min_linear_acceleration>-2</min_linear_acceleration>
@@ -188,5 +188,5 @@
       <!-- Changed the height of 2D LiDAR to avoid the problem of Gazebo -->
       <origin rpy="0 0 ${PI / 2.0}"
-              xyz="0.156 0 0.1549" />
+              xyz="0.156 0 0.1049" />
     </joint>
     <link name="laser_frame" />
@@ -382,23 +382,23 @@
       <parent link="base_link"/>
       <child link="caster1_link"/>
-      <origin xyz="0.19 0.075 0.01" rpy="0 0 0"/>
+      <origin xyz="0.19 0.075 0.0" rpy="0 0 0"/>
     </joint>
     <link name="caster1_link">
       <visual>
         <geometry>
-          <sphere radius="0.01"/>
-        </geometry>
-        <material name="tire" />
-      </visual>
-      <collision>
-        <geometry>
-          <sphere radius="0.01"/>
-        </geometry>
-      </collision>
-      <inertial>
-        <mass value="0.01" />
-        <inertia ixx="${(2/5) * 0.01 * 0.01 * 0.01}" ixy="0.0" ixz="0.0"
-                 iyy="${(2/5) * 0.01 * 0.01 * 0.01}" iyz="0.0"
-                 izz="${(2/5) * 0.01 * 0.01 * 0.01}" />
+          <sphere radius="0.005"/>
+        </geometry>
+        <material name="tire" />
+      </visual>
+      <collision>
+        <geometry>
+          <sphere radius="0.005"/>
+        </geometry>
+      </collision>
+      <inertial>
+        <mass value="0.005" />
+        <inertia ixx="${(2/5) * 0.005 * 0.005 * 0.005}" ixy="0.0" ixz="0.0"
+                 iyy="${(2/5) * 0.005 * 0.005 * 0.005}" iyz="0.0"
+                 izz="${(2/5) * 0.005 * 0.005 * 0.005}" />
       </inertial>
     </link>
@@ -416,23 +416,23 @@
       <parent link="base_link"/>
       <child link="caster2_link"/>
-      <origin xyz="0.19 -0.075 0.01" rpy="0 0 0"/>
+      <origin xyz="0.19 -0.075 0.0" rpy="0 0 0"/>
     </joint>
     <link name="caster2_link">
       <visual>
         <geometry>
-          <sphere radius="0.01"/>
-        </geometry>
-        <material name="tire" />
-      </visual>
-      <collision>
-        <geometry>
-          <sphere radius="0.01"/>
-        </geometry>
-      </collision>
-      <inertial>
-        <mass value="0.01" />
-        <inertia ixx="${(2/5) * 0.01 * 0.01 * 0.01}" ixy="0.0" ixz="0.0"
-                 iyy="${(2/5) * 0.01 * 0.01 * 0.01}" iyz="0.0"
-                 izz="${(2/5) * 0.01 * 0.01 * 0.01}" />
+          <sphere radius="0.005"/>
+        </geometry>
+        <material name="tire" />
+      </visual>
+      <collision>
+        <geometry>
+          <sphere radius="0.005"/>
+        </geometry>
+      </collision>
+      <inertial>
+        <mass value="0.005" />
+        <inertia ixx="${(2/5) * 0.005 * 0.005 * 0.005}" ixy="0.0" ixz="0.0"
+                 iyy="${(2/5) * 0.005 * 0.005 * 0.005}" iyz="0.0"
+                 izz="${(2/5) * 0.005 * 0.005 * 0.005}" />
       </inertial>
     </link>
